Commit message: bugfix: camera position colliding with robot

File: catkin_ws/src/universal_robot/ur_e_description/urdf/ur10e.urdf.xacro (robot description, xacro)
@@ -319,5 +319,5 @@
     <joint name="camera_joint" type="fixed">
     <axis xyz="0 1 0" />
-    <origin xyz="-0.02 0.0 0.055" rpy="0 0 0"/>
+    <origin xyz="0.005 0.0 0.055" rpy="0 0 0"/>
     <parent link="${prefix}ee_link"/>
     <child link="camera_link"/>
