Commit message: Added camera to UR10 in Gazebo

File: catkin_ws/src/universal_robot/ur_e_description/urdf/common.gazebo.xacro (robot description, xacro)
@@ -21,3 +21,43 @@
 -->
   </gazebo>
+  <!-- camera -->
+  <gazebo reference="camera_link">
+    <sensor type="camera" name="camera1">
+      <update_rate>30.0</update_rate>
+      <camera name="head">
+        <horizontal_fov>1.3962634</horizontal_fov>
+        <image>
+          <width>800</width>
+          <height>800</height>
+          <format>R8G8B8</format>
+        </image>
+        <clip>
+          <near>0.02</near>
+          <far>300</far>
+        </clip>
+        <noise>
+          <type>gaussian</type>
+          <!-- Noise is sampled independently per pixel on each frame.
+               That pixel's noise value is added to each of its color
+               channels, which at that point lie in the range [0,1]. -->
+          <mean>0.0</mean>
+          <stddev>0.007</stddev>
+        </noise>
+      </camera>
+      <plugin name="camera_controller" filename="libgazebo_ros_camera.so">
+        <alwaysOn>true</alwaysOn>
+        <updateRate>0.0</updateRate>
+        <cameraName>ur10e/camera1</cameraName>
+        <imageTopicName>image_raw</imageTopicName>
+        <cameraInfoTopicName>camera_info</cameraInfoTopicName>
+        <frameName>camera_link</frameName>
+        <hackBaseline>0.07</hackBaseline>
+        <distortionK1>0.0</distortionK1>
+        <distortionK2>0.0</distortionK2>
+        <distortionK3>0.0</distortionK3>
+        <distortionT1>0.0</distortionT1>
+        <distortionT2>0.0</distortionT2>
+      </plugin>
+    </sensor>
+  </gazebo>
 </robot>

File: catkin_ws/src/universal_robot/ur_e_description/urdf/ur10e.urdf.xacro (robot description, xacro)
@@ -34,4 +34,6 @@
     <xacro:property name="wrist_2_mass" value="1.96" />
     <xacro:property name="wrist_3_mass" value="0.202" />
+    <xacro:property name="height3" value="1" /> <!-- Link 3 -->
+    <xacro:property name="camera_link" value="0.02" /> <!-- Size of square 'camera' box -->
     <!-- These parameters are borrowed from the urcontrol.conf file
         but are not verified for the correct permutation.
@@ -315,4 +317,31 @@
       </collision>
     </link>
+    <joint name="camera_joint" type="fixed">
+    <axis xyz="0 1 0" />
+    <origin xyz="-0.02 0.0 0.055" rpy="0 0 0"/>
+    <parent link="${prefix}ee_link"/>
+    <child link="camera_link"/>
+  </joint>
+  <!-- Camera -->
+  <link name="camera_link">
+    <collision>
+      <origin xyz="0 0 0" rpy="0 0 0"/>
+      <geometry>
+    <box size="${camera_link} ${camera_link} ${camera_link}"/>
+      </geometry>
+    </collision>
+    <visual>
+      <origin xyz="0 0 0" rpy="0 0 0"/>
+      <geometry>
+    <box size="${camera_link} ${camera_link} ${camera_link}"/>
+      </geometry>
+      <material name="LightGrey"/>
+    </visual>
+    <inertial>
+      <mass value="1e-5" />
+      <origin xyz="0 0 0" rpy="0 0 0"/>
+      <inertia ixx="1e-6" ixy="0" ixz="0" iyy="1e-6" iyz="0" izz="1e-6" />
+    </inertial>
+  </link>
     <xacro:ur_arm_transmission prefix="${prefix}" />
     <xacro:ur_arm_gazebo prefix="${prefix}" />

File: catkin_ws/src/universal_robot/ur_e_description/urdf/ur10e_joint_limited_robot.urdf.xacro (robot description, xacro)
@@ -8,5 +8,5 @@
   <!-- arm -->
   <xacro:ur10e_robot prefix="" joint_limited="true"
-		 shoulder_pan_lower_limit="${-pi}" shoulder_pan_upper_limit="${pi}"
+		 shoulder_pan_lower_limit="${-2*pi}" shoulder_pan_upper_limit="${2*pi}"
 		 shoulder_lift_lower_limit="${-pi}" shoulder_lift_upper_limit="${pi}"
 		 elbow_joint_lower_limit="${-pi}" elbow_joint_upper_limit="${pi}"

Commit message: feat: move point cloud along quaternions (I do not want to do this math again)

File: catkin_ws/src/universal_robot/ur_e_description/urdf/common.gazebo.xacro (robot description, xacro)
@@ -57,5 +57,5 @@
             <depthImageCameraInfoTopicName>depth/camera_info</depthImageCameraInfoTopicName>
             <pointCloudTopicName>depth/points</pointCloudTopicName>
-            <frameName>camera_link</frameName>
+            <frameName>camera_frame_optical</frameName>
             <pointCloudCutoff>0.5</pointCloudCutoff>
             <pointCloudCutoffMax>3.0</pointCloudCutoffMax>

File: catkin_ws/src/universal_robot/ur_e_description/urdf/ur10e.urdf.xacro (robot description, xacro)
@@ -317,4 +317,10 @@
       </collision>
     </link>
+    <joint name="camera_optical_joint" type="fixed">
+    <origin xyz="0 0 0" rpy="-1.5708 0 -1.5708"/>
+    <parent link="camera_link"/>
+    <child link="camera_frame_optical"/>
+    </joint>
+    <link name="camera_frame_optical"/>
     <joint name="camera_joint" type="fixed">
     <axis xyz="0 1 0" />
